File: DriveBayLCD.sch (EAGLE design)
At the start: 31 parts, among them J1 AVR_SPI_PRG_6PTH, U1 ATMEGA32U2-AU, U2 2N7002, X1 22-23-2041

Commit message: Added mising 22 ohms line resistors
Parts:
- added R10, R11: 22, resistor:R-EU_R0805
Connections:
- new net N$125: R10.1, U1.D+
- new net N$126: R11.1, U1.D-
- net D+: now also R10.2; no longer U1.D+
- net D-: now also R11.2; no longer U1.D-
Changed lines of the file:
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@@
 <part name="R8" library="resistor" deviceset="R-EU_" device="R0805"/>
 <part name="R9" library="resistor" deviceset="R-EU_" device="R0805" value="10"/>
+<part name="R10" library="resistor" deviceset="R-EU_" device="R0805" value="22"/>
+<part name="R11" library="resistor" deviceset="R-EU_" device="R0805" value="22"/>
 </parts>
 <sheets>
@@
 <instance part="R8" gate="G$1" x="25.4" y="200.66"/>
 <instance part="R9" gate="G$1" x="233.68" y="60.96" rot="R180"/>
+<instance part="R10" gate="G$1" x="68.58" y="45.72" smashed="yes" rot="R180">
+<attribute name="NAME" x="67.818" y="49.0474" size="1.778" layer="95" rot="R180"/>
+<attribute name="VALUE" x="74.422" y="48.768" size="1.778" layer="96" rot="R180"/>
+</instance>
+<instance part="R11" gate="G$1" x="68.58" y="43.18" smashed="yes" rot="R180">
+<attribute name="NAME" x="73.66" y="41.402" size="1.778" layer="95" rot="R180"/>
+<attribute name="VALUE" x="67.31" y="41.402" size="1.778" layer="96" rot="R180"/>
+</instance>
 </instances>
 <busses>
@@
 </segment>
 <segment>
-<pinref part="U1" gate="A" pin="D+"/>
-<wire x1="76.2" y1="45.72" x2="73.66" y2="45.72" width="0.1524" layer="91"/>
-<label x="73.66" y="45.72" size="1.27" layer="95" rot="R180" xref="yes"/>
+<pinref part="R10" gate="G$1" pin="2"/>
+<wire x1="63.5" y1="45.72" x2="60.96" y2="45.72" width="0.1524" layer="91"/>
+<label x="60.96" y="45.72" size="1.27" layer="95" rot="R180" xref="yes"/>
 </segment>
 </net>
@@
 </segment>
 <segment>
-<pinref part="U1" gate="A" pin="D-"/>
-<wire x1="76.2" y1="43.18" x2="73.66" y2="43.18" width="0.1524" layer="91"/>
-<label x="73.66" y="43.18" size="1.27" layer="95" rot="R180" xref="yes"/>
+<pinref part="R11" gate="G$1" pin="2"/>
+<wire x1="63.5" y1="43.18" x2="60.96" y2="43.18" width="0.1524" layer="91"/>
+<label x="60.96" y="43.18" size="1.27" layer="95" rot="R180" xref="yes"/>
 </segment>
 </net>
@@
 </segment>
 </net>
+<net name="N$126" class="0">
+<segment>
+<pinref part="U1" gate="A" pin="D-"/>
+<wire x1="76.2" y1="43.18" x2="73.66" y2="43.18" width="0.1524" layer="91"/>
+<pinref part="R11" gate="G$1" pin="1"/>
+</segment>
+</net>
+<net name="N$125" class="0">
+<segment>
+<pinref part="U1" gate="A" pin="D+"/>
+<wire x1="76.2" y1="45.72" x2="73.66" y2="45.72" width="0.1524" layer="91"/>
+<pinref part="R10" gate="G$1" pin="1"/>
+</segment>
+</net>
